Commit message: Changed smarc_auvs refs to smarc_private_auvs

File: robots/lolo_auv_default.urdf.xacro (robot description, xacro)
@@ -16,5 +16,5 @@
   <xacro:arg name="namespace" default="lolo_auv"/>
   <!-- Include the UUV macro file -->
-  <xacro:include filename="$(find smarc_auvs)/models/lolo_auv/urdf/lolo_auv_base.urdf.xacro"/>
+  <xacro:include filename="$(find smarc_private_auvs)/models/lolo_auv/urdf/lolo_auv_base.urdf.xacro"/>
   <!-- Create the romulus -->
   <xacro:lolo_auv_base namespace="$(arg namespace)" debug="$(arg debug)"/>

File: urdf/lolo_auv_base.urdf.xacro (robot description, xacro)
@@ -27,8 +27,8 @@
   <xacro:property name="cob" value="0 0 0.0196"/>
   <xacro:property name="rho" value="1025.0"/>
-  <xacro:property name="visual_mesh_file" value="file://$(find smarc_auvs)/models/lolo_auv/mesh/lolo.dae"/>
-  <xacro:property name="prop_mesh_file" value="file://$(find smarc_auvs)/models/lolo_auv/mesh/propeller.dae"/>
-  <xacro:property name="fin_mesh_file" value="file://$(find smarc_auvs)/models/lolo_auv/mesh/fin.dae"/>
-  <xacro:property name="back_fin_mesh_file" value="file://$(find smarc_auvs)/models/lolo_auv/mesh/back_fin.dae"/>
+  <xacro:property name="visual_mesh_file" value="file://$(find smarc_private_auvs)/models/lolo_auv/mesh/lolo.dae"/>
+  <xacro:property name="prop_mesh_file" value="file://$(find smarc_private_auvs)/models/lolo_auv/mesh/propeller.dae"/>
+  <xacro:property name="fin_mesh_file" value="file://$(find smarc_private_auvs)/models/lolo_auv/mesh/fin.dae"/>
+  <xacro:property name="back_fin_mesh_file" value="file://$(find smarc_private_auvs)/models/lolo_auv/mesh/back_fin.dae"/>
   <!-- Fin snippet -->
   <xacro:macro name="fin_macro" params="namespace fin_id *origin">
