Commit message: Added the new forward-looking sonar to lolo

File: urdf/lolo_auv_base.urdf.xacro (robot description, xacro)
@@ -345,4 +345,21 @@
       </visual>
     </xacro:multibeam_intensity_sonar>
+	<!-- Forward looking sonar -->
+	<xacro:forward_looking_sonar
+      namespace="${namespace}"
+      suffix="down"
+      parent_link="${namespace}/base_link"
+      topic="forward_sonar"
+      mass="0.015"
+      update_rate="10"
+      samples="100"
+	  fov="1.54719755"
+	  width="1040"
+	  height="480">
+      <inertia ixx="0.00001" ixy="0.0" ixz="0.0" iyy="0.00001" iyz="0.0" izz="0.00001" />
+      <origin xyz="1.0 0 -0.3" rpy="0 ${0.2*pi} 0" />
+      <visual>
+      </visual>
+    </xacro:forward_looking_sonar>
     <!-- RPT
     <xacro:default_rpt namespace="${namespace}" parent_link="${namespace}/base_link">

Commit message: Added MBES plugin to LoLo and renamed SSS macro to side_scan_sonar

File: urdf/lolo_auv_base.urdf.xacro (robot description, xacro)
@@ -308,5 +308,5 @@
     </xacro:dvl_plugin_macro>
     <!-- Side scan sonar left -->
-    <xacro:multibeam_intensity_sonar
+    <xacro:side_scan_sonar
       namespace="${namespace}"
       suffix="left"
@@ -325,7 +325,7 @@
       <visual>
       </visual>
-    </xacro:multibeam_intensity_sonar>
+    </xacro:side_scan_sonar>
     <!-- Side scan sonar right -->
-    <xacro:multibeam_intensity_sonar
+    <xacro:side_scan_sonar
       namespace="${namespace}"
       suffix="right"
@@ -344,7 +344,26 @@
       <visual>
       </visual>
+    </xacro:side_scan_sonar>
+    <!-- Multibeam sonar -->
+    <xacro:multibeam_intensity_sonar
+      namespace="${namespace}"
+      suffix="down"
+      parent_link="${namespace}/base_link"
+      topic="mbes_laser"
+      mass="0.015"
+      update_rate="5"
+      samples="135"
+      fov="${3.0*pi/4.0}"
+      range_min="1.0"
+      range_max="200.0"
+      range_stddev="0.027"
+      mesh="">
+      <inertia ixx="0.00001" ixy="0.0" ixz="0.0" iyy="0.00001" iyz="0.0" izz="0.00001" />
+      <origin xyz="0.0 0.0 -0.3" rpy="0.0 ${pi/2.0} 0.0" />
+      <visual>
+      </visual>
     </xacro:multibeam_intensity_sonar>
-	<!-- Forward looking sonar -->
-	<xacro:forward_looking_sonar
+  	<!-- Forward looking sonar -->
+  	<xacro:forward_looking_sonar
       namespace="${namespace}"
       suffix="down"

Commit message: Moved fls a bit

File: urdf/lolo_auv_base.urdf.xacro (robot description, xacro)
@@ -358,5 +358,5 @@
 	  height="480">
       <inertia ixx="0.00001" ixy="0.0" ixz="0.0" iyy="0.00001" iyz="0.0" izz="0.00001" />
-      <origin xyz="1.0 0 -0.3" rpy="0 ${0.2*pi} 0" />
+      <origin xyz="0.83 0 -0.22" rpy="0 ${0.2*pi} 0" />
       <visual>
       </visual>

Commit message: LoLo xacro file cleaned for dryrun demo

File: urdf/lolo_auv_base.urdf.xacro (robot description, xacro)
@@ -307,44 +307,6 @@
       <origin xyz="0.4785 0.0 -0.0825" rpy="0 ${0.5*pi} 0" />
     </xacro:dvl_plugin_macro>
-    <!-- Side scan sonar left -->
-    <xacro:multibeam_intensity_sonar
-      namespace="${namespace}"
-      suffix="left"
-      parent_link="${namespace}/base_link"
-      topic="sss_left"
-      mass="0.015"
-      update_rate="5"
-      samples="100"
-      fov="${pi/3.0}"
-      range_min="1.0"
-      range_max="200.0"
-      range_stddev="0.027"
-      mesh="">
-      <inertia ixx="0.00001" ixy="0.0" ixz="0.0" iyy="0.00001" iyz="0.0" izz="0.00001" />
-      <origin xyz="0.41225 0.1498 -0.04615" rpy="${0.5*pi} ${-5*d2r+pi/3.0} ${0.5*pi}" />
-      <visual>
-      </visual>
-    </xacro:multibeam_intensity_sonar>
-    <!-- Side scan sonar right -->
-    <xacro:multibeam_intensity_sonar
-      namespace="${namespace}"
-      suffix="right"
-      parent_link="${namespace}/base_link"
-      topic="sss_right"
-      mass="0.015"
-      update_rate="5"
-      samples="100"
-      fov="${pi/3.0}"
-      range_min="1.0"
-      range_max="200.0"
-      range_stddev="0.027"
-      mesh="">
-      <inertia ixx="0.00001" ixy="0.0" ixz="0.0" iyy="0.00001" iyz="0.0" izz="0.00001" />
-      <origin xyz="0.41225 -0.1498 -0.04615" rpy="${0.5*pi} ${-5*d2r+pi/3.0} ${-0.5*pi}" />
-      <visual>
-      </visual>
-    </xacro:multibeam_intensity_sonar>
 	<!-- Forward looking sonar -->
-	<xacro:forward_looking_sonar
+<!-- 	<xacro:forward_looking_sonar
       namespace="${namespace}"
       suffix="down"
@@ -361,13 +323,5 @@
       <visual>
       </visual>
-    </xacro:forward_looking_sonar>
-    <!-- RPT
-    <xacro:default_rpt namespace="${namespace}" parent_link="${namespace}/base_link">
-      <origin xyz="0 0 0" rpy="0 0 0"/>
-    </xacro:default_rpt>  -->
-    <!-- Pressure
-    <xacro:default_pressure namespace="${namespace}" parent_link="${namespace}/base_link">
-      <origin xyz="0 0 0" rpy="0 0 0"/>
-    </xacro:default_pressure>  -->
+    </xacro:forward_looking_sonar> -->
     <!-- IMU  -->
     <xacro:default_imu namespace="${namespace}" parent_link="${namespace}/base_link">

Commit message: LoLo with basic cameras only

File: urdf/lolo_auv_base.urdf.xacro (robot description, xacro)
@@ -299,5 +299,5 @@
     </gazebo>
     <!-- DVL sensor -->
-    <xacro:dvl_plugin_macro
+<!--     <xacro:dvl_plugin_macro
       namespace="${namespace}"
       suffix=""
@@ -306,5 +306,5 @@
       scale="0.62">
       <origin xyz="0.4785 0.0 -0.0825" rpy="0 ${0.5*pi} 0" />
-    </xacro:dvl_plugin_macro>
+    </xacro:dvl_plugin_macro> -->
 	<!-- Forward looking sonar -->
     <!-- <xacro:forward_looking_sonar
@@ -325,7 +325,26 @@
     </xacro:forward_looking_sonar> -->
     <!-- IMU  -->
-    <xacro:default_imu namespace="${namespace}" parent_link="${namespace}/base_link">
+<!--     <xacro:default_imu namespace="${namespace}" parent_link="${namespace}/base_link">
       <origin xyz="0 0 0" rpy="0 0 0"/>
-    </xacro:default_imu>
+    </xacro:default_imu> -->
+        <!-- Multibeam sonar -->
+<!--     <xacro:multibeam_intensity_sonar
+      namespace="${namespace}"
+      suffix="down"
+      parent_link="${namespace}/base_link"
+      topic="mbes_laser"
+      mass="0.015"
+      update_rate="15"
+      samples="235"
+      fov="${4.0*pi/6.0}"
+      range_min="1.0"
+      range_max="200.0"
+      range_stddev="0.027"
+      mesh="">
+      <inertia ixx="0.00001" ixy="0.0" ixz="0.0" iyy="0.00001" iyz="0.0" izz="0.00001" />
+      <origin xyz="0.0 0.0 -0.3" rpy="0.0 ${pi/2.0} 0.0" />
+      <visual>
+      </visual>
+    </xacro:multibeam_intensity_sonar> -->
 	<!-- Mount a camera -->
     <xacro:regular_camera_plugin_macro
