Commit message: added decals to lolo, check the blend file for modifications

File: lolo_auv_sim/urdf/lolo_auv_base.urdf.xacro (robot description, xacro)
@@ -31,4 +31,5 @@
   <xacro:property name="fin_mesh_file" value="file://$(find lolo_auv_sim)/mesh/fin.dae"/>
   <xacro:property name="back_fin_mesh_file" value="file://$(find lolo_auv_sim)/mesh/back_fin.dae"/>
+  <xacro:property name="decals_mesh_file" value="file://$(find lolo_auv_sim)/mesh/decals.dae"/>
   <!-- Fin snippet -->
   <xacro:macro name="fin_macro" params="namespace fin_id *origin">
@@ -128,4 +129,17 @@
                  izz="3.45" />
       </inertial>
+    </link>
+    <!-- Create a floating decal -->
+    <joint name="base_link_to_decals" type="fixed">
+        <parent link="${namespace}/base_link"/>
+        <child link="${namespace}/decals"/>
+    </joint>
+    <link name="${namespace}/decals">
+      <visual>
+        <origin xyz="0 0 0" rpy="0 0 0"/>
+        <geometry>
+          <mesh filename="${decals_mesh_file}" scale="1 1 1" />
+        </geometry>
+      </visual>
     </link>
     <!-- Set up hydrodynamic plugin -->
