Commit message: Update meshes and robot description to match current status of real lolo

File: lolo_description/urdf/actuators.xacro (robot description, xacro)
@@ -4,6 +4,7 @@
   <xacro:property name="prop_strb_mesh_file" value="file://$(find lolo_description)/mesh/lolo_strb_propeller.dae"/>
   <xacro:property name="rudder_mesh_file" value="file://$(find lolo_description)/mesh/lolo_rudder.dae"/>
-  <xacro:property name="elevon_port_mesh_file" value="file://$(find lolo_description)/mesh/lolo_port_elevon.dae"/>
-  <xacro:property name="elevon_strb_mesh_file" value="file://$(find lolo_description)/mesh/lolo_strb_elevon.dae"/>
+  <!--<xacro:property name="elevon_port_mesh_file" value="file://$(find lolo_description)/mesh/lolo_port_elevon.dae"/>-->
+  <!--<xacro:property name="elevon_strb_mesh_file" value="file://$(find lolo_description)/mesh/lolo_strb_elevon.dae"/>-->
+  <xacro:property name="elevon_mesh_file" value="file://$(find lolo_description)/mesh/lolo_elevon.dae"/>
   <xacro:property name="elevator_mesh_file" value="file://$(find lolo_description)/mesh/lolo_elevator.dae"/>
   <xacro:thruster_module_first_order_basic_fcn_macro
@@ -12,5 +13,5 @@
       dyn_time_constant="0.05"
       rotor_constant="0.0006279">
-    <origin xyz="-0.9056 0.2754 0.013678" rpy="0 0 0" />
+      <origin xyz="-0.9056 0.2754 0.013678" rpy="0 0 ${pi}" />
   </xacro:thruster_module_first_order_basic_fcn_macro>
   <xacro:thruster_module_first_order_basic_fcn_macro
@@ -28,12 +29,12 @@
     <origin xyz="-0.3278 0.253 0.129" rpy="0 0 0" />
   </xacro:fin_macro>
-  <xacro:fin_macro namespace="${namespace}" fin_id="2" mesh_filename="${elevon_strb_mesh_file}">
-    <origin xyz="-0.3733 -0.4035 0.01349" rpy="0 0 -0.19652" />
+  <xacro:fin_macro namespace="${namespace}" fin_id="2" mesh_filename="${elevon_mesh_file}">
+      <origin xyz="-0.3733 -0.4035 0.01349" rpy="${0.5 * pi} 0 0" />
   </xacro:fin_macro>
-  <xacro:fin_macro namespace="${namespace}" fin_id="3" mesh_filename="${elevon_port_mesh_file}">
-    <origin xyz="-0.3733 0.4035 0.01349" rpy="0 0 0.19652" />
+  <xacro:fin_macro namespace="${namespace}" fin_id="3" mesh_filename="${elevon_mesh_file}">
+      <origin xyz="-0.3733 0.4035 0.01349" rpy="${-0.5 * pi} 0 0" />
   </xacro:fin_macro>
   <xacro:fin_macro namespace="${namespace}" fin_id="4" mesh_filename="${elevator_mesh_file}">
-    <origin xyz="-0.6476 0.0 0.0135" rpy="0 0 0" />
+      <origin xyz="-0.6476 0.0 0.0135" rpy="${0.5 * pi} 0 0" />
   </xacro:fin_macro>
 </robot>
