Commit message: Added links for sensors in the tree

File: lolo_description/urdf/lolo_auv.urdf.xacro (robot description, xacro)
@@ -13,4 +13,9 @@
     </visual>
   </link>
+  <link name="$(arg robot_namespace)/dvl_link"/>
+  <link name="$(arg robot_namespace)/compass_link"/>
+  <link name="$(arg robot_namespace)/fls_link"/>
+  <link name="$(arg robot_namespace)/imu_link"/>
+  <link name="$(arg robot_namespace)/pressure_link"/>
   <link name="$(arg robot_namespace)/elevator">
     <visual>
@@ -165,3 +170,28 @@
     <limit effort="0" lower="0" upper="0" velocity="0"/>
   </joint>
+  <joint name="$(arg robot_namespace)/dvl_joint" type="fixed">
+    <origin xyz="0 0 0" rpy="0 0 0" />
+    <parent link="$(arg robot_namespace)/base_link"/>
+    <child link="$(arg robot_namespace)/dvl_link"/>
+  </joint>
+  <joint name="$(arg robot_namespace)/compass_joint" type="fixed">
+    <origin xyz="0 0 0" rpy="0 0 0" />
+    <parent link="$(arg robot_namespace)/base_link"/>
+    <child link="$(arg robot_namespace)/compass_link"/>
+  </joint>
+  <joint name="$(arg robot_namespace)/fls_joint" type="fixed">
+    <origin xyz="0 0 0" rpy="0 0 0" />
+    <parent link="$(arg robot_namespace)/base_link"/>
+    <child link="$(arg robot_namespace)/fls_link"/>
+  </joint>
+  <joint name="$(arg robot_namespace)/imu_joint" type="fixed">
+    <origin xyz="0 0 0" rpy="0 0 0" />
+    <parent link="$(arg robot_namespace)/base_link"/>
+    <child link="$(arg robot_namespace)/imu_link"/>
+  </joint>
+  <joint name="$(arg robot_namespace)/pressure_joint" type="fixed">
+    <origin xyz="0 0 0" rpy="0 0 0" />
+    <parent link="$(arg robot_namespace)/base_link"/>
+    <child link="$(arg robot_namespace)/pressure_link"/>
+  </joint>
 </robot>

Commit message: Added gps link also

File: lolo_description/urdf/lolo_auv.urdf.xacro (robot description, xacro)
@@ -18,4 +18,5 @@
   <link name="$(arg robot_namespace)/imu_link"/>
   <link name="$(arg robot_namespace)/pressure_link"/>
+  <link name="$(arg robot_namespace)/gps_link"/>
   <link name="$(arg robot_namespace)/elevator">
     <visual>
@@ -195,3 +196,8 @@
     <child link="$(arg robot_namespace)/pressure_link"/>
   </joint>
+  <joint name="$(arg robot_namespace)/gps_joint" type="fixed">
+    <origin xyz="0 0 0" rpy="0 0 0" />
+    <parent link="$(arg robot_namespace)/base_link"/>
+    <child link="$(arg robot_namespace)/gps_link"/>
+  </joint>
 </robot>

Commit message: updated lolo description from a long time ago

File: lolo_description/urdf/lolo_auv.urdf.xacro (robot description, xacro)
@@ -23,4 +23,5 @@
   <link name="$(arg robot_namespace)/gps_link"/>
   <link name="$(arg robot_namespace)/mbes_link"/>
+  <link name="$(arg robot_namespace)/enu/mbes_link"/>
   <link name="$(arg robot_namespace)/usbl_link"/>
   <link name="$(arg robot_namespace)/elevator">
@@ -177,4 +178,9 @@
     <child link="$(arg robot_namespace)/mbes_link"/>
   </joint>
+  <joint name="$(arg robot_namespace)/enu/mbes_joint" type="fixed">
+    <origin xyz="2.523 0.0155 -0.302" rpy="0 0 0" />
+    <parent link="$(arg robot_namespace)/base_link"/>
+    <child link="$(arg robot_namespace)/enu/mbes_link"/>
+  </joint>
   <joint name="$(arg robot_namespace)/usbl_joint" type="fixed">
     <origin xyz="0.389 0.002 0.337" rpy="0 0 0" />
